Commit message: Update wheel.xacro

File: steer_bot_description/urdf/wheel.xacro (robot description, xacro)
@@ -49,5 +49,5 @@
       <parent link="${parent}_link"/>
       <child link="${name}_steer_link"/>
-      <origin xyz="${base_length/2-axle_offset} 0 ${steer_height}" rpy="0 0 0"/>
+      <origin xyz="0 0 ${steer_height}" rpy="0 0 0"/>
       <axis xyz="0 0 1"/>
       <limit effort="${steer_effort}"

Commit message: Add files via upload

File: steer_bot_description/urdf/wheel.xacro (robot description, xacro)
@@ -165,6 +165,6 @@
     </gazebo>
   </xacro:macro>
-  <!-- Car steering model rear wheel links (left/right) -->
-  <xacro:macro name="rear_wheel_lr"
+  <!-- Bicycle model rear wheel link (required for steer_drive_controller) -->
+  <xacro:macro name="rear_wheel"
     params="
       name
@@ -180,5 +180,5 @@
           <cylinder radius="${wheel_radius}" length="${wheel_thickness}"/>
         </geometry>
-        <material name="red" />
+        <material name="yellow" />
       </visual>
       <collision>
@@ -210,4 +210,93 @@
     </transmission>
     <gazebo reference="${name}_wheel_link">
+      <material>Gazebo/Yellow</material>
+    </gazebo>
+  </xacro:macro>
+  <!-- Bicycle model front wheel link (passive - no transmission) -->
+  <xacro:macro name="front_wheel"
+    params="
+      name
+      parent
+      wheel_radius
+      wheel_thickness
+      wheel_mass
+      *origin">
+    <link name="${name}_wheel_link">
+      <visual>
+        <origin xyz="0 0 0" rpy="0 0 0"/>
+        <geometry>
+          <cylinder radius="${wheel_radius}" length="${wheel_thickness}"/>
+        </geometry>
+        <material name="yellow" />
+      </visual>
+      <collision>
+        <origin xyz="0 0 0" rpy="0 0 0"/>
+        <geometry>
+          <cylinder radius="${wheel_radius}" length="${wheel_thickness}"/>
+        </geometry>
+      </collision>
+      <xacro:solid_cylinder_inertial
+          rpy="0 0 0" xyz="0 0 0"
+          mass="${wheel_mass}"
+          radius="${wheel_radius}" length="${wheel_thickness}" />
+    </link>
+    <joint name="${name}_wheel_joint" type="continuous">
+      <parent link="${parent}_link"/>
+      <child link="${name}_wheel_link"/>
+      <xacro:insert_block name="origin"/>
+      <axis xyz="0 0 1"/>
+    </joint>
+    <gazebo reference="${name}_wheel_link">
+      <material>Gazebo/Yellow</material>
+    </gazebo>
+    <gazebo reference="${name}_wheel_joint">
+      <provideFeedback>true</provideFeedback>
+    </gazebo>
+  </xacro:macro>
+  <!-- Car steering model rear wheel links (left/right) -->
+  <xacro:macro name="rear_wheel_lr"
+    params="
+      name
+      parent
+      wheel_radius
+      wheel_thickness
+      wheel_mass
+      *origin">
+    <link name="${name}_wheel_link">
+      <visual>
+        <origin xyz="0 0 0" rpy="0 0 0"/>
+        <geometry>
+          <cylinder radius="${wheel_radius}" length="${wheel_thickness}"/>
+        </geometry>
+        <material name="red" />
+      </visual>
+      <collision>
+        <origin xyz="0 0 0" rpy="0 0 0"/>
+        <geometry>
+          <cylinder radius="${wheel_radius}" length="${wheel_thickness}"/>
+        </geometry>
+      </collision>
+      <xacro:solid_cylinder_inertial
+          rpy="0 0 0" xyz="0 0 0"
+          mass="${wheel_mass}"
+          radius="${wheel_radius}" length="${wheel_thickness}" />
+    </link>
+    <joint name="${name}_wheel_joint" type="continuous">
+      <parent link="${parent}_link"/>
+      <child link="${name}_wheel_link"/>
+      <xacro:insert_block name="origin"/>
+      <axis xyz="0 0 1"/>
+    </joint>
+    <transmission name="${name}_wheel_joint_trans">
+      <type>transmission_interface/SimpleTransmission</type>
+      <actuator name="${name}_wheel_joint_motor">
+        <mechanicalReduction>1</mechanicalReduction>
+        <hardwareInterface>hardware_interface/VelocityJointInterface</hardwareInterface>
+      </actuator>
+      <joint name="${name}_wheel_joint">
+        <hardwareInterface>hardware_interface/VelocityJointInterface</hardwareInterface>
+      </joint>
+    </transmission>
+    <gazebo reference="${name}_wheel_link">
       <material>Gazebo/Red</material>
     </gazebo>
